File: odins-eye-pcb/odins-eye-pcb.kicad_pcb (KiCad board)
At the start: 4 copper layers, 105.5 x 50 mm, 9 parts, among them J2 TF-LUNA CONNECTOR, J3 POWER USB C

Commit message: Add odins-eye v1.1
Parts:
- added J4: GYROSCOPE-CONNECTOR, Connector_PinSocket_2.54mm:PinSocket_1x08_P2.54mm_Vertical, B.Cu at (162.0, 75.5)
- J3: value POWER USB C -> POWER USB-C
- Raspberry Pi Zero 2 W: renamed from Raspberry Pi Zero 2 W Header
Connections:
- J2 pad 2: /RXD -> /SDA
- J2 pad 3: /TXD -> /SCL
- J2 pad 5: unconnected-(J2-Pin_5-Pad5) -> GND
- Raspberry Pi Zero 2 W pad 10: /TXD -> unconnected-(U1-RXD0-Pad10)
- Raspberry Pi Zero 2 W pad 3: unconnected-(U1-SDA1-Pad3) -> /SDA
- Raspberry Pi Zero 2 W pad 5: unconnected-(U1-SCL1-Pad5) -> /SCL
- Raspberry Pi Zero 2 W pad 8: /RXD -> unconnected-(U1-TXD0-Pad8)
Routing:
- net /SCL: track 0.00 -> 39.9 mm, vias 0 -> 2
- net /SDA: track 0.00 -> 36.6 mm
- net +3V3: track 50.4 -> 73.8 mm
- net GND: track 0.00 -> 15.8 mm
- net /RXD: track 14.1 -> 0.00 mm
- net /TXD: track 13.3 -> 0.00 mm, vias 1 -> 0
Other:
- board size 105.5 x 50 mm -> 102 x 50 mm

Commit message: Update arduino code
Parts:
- removed the G*** at (168.5, 112.5)
- added G***: LOGO, LOGO, F.Cu at (168.1, 111.8)
- added G***: LOGO, LOGO, B.Cu at (167.4, 112.3)

Commit message: Update 3D printed case
Other:
- board size 102 x 50 mm -> 102 x 55 mm
Changed lines of the file:
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@@
 		)
+	)
+	(gr_circle
+		(center 195.1 86)
+		(end 195.1 84.9)
+		(stroke
+			(width 0.0381)
+			(type default)
+		)
+		(fill no)
+		(layer "Edge.Cuts")
 	)
 	(gr_line
-		(start 97.375 69.525)
-		(end 199.375 69.525)
+		(start 97.375 64.525)
+		(end 199.375 64.525)
 		(stroke
 			(width 0.0381)
@@
 		(layer "Edge.Cuts")
 	)
-	(gr_line
-		(start 199.375 119.525)
-		(end 199.375 69.525)
+	(gr_circle
+		(center 195.1 73.5)
+		(end 195.1 72.4)
 		(stroke
 			(width 0.0381)
 			(type default)
 		)
+		(fill no)
+		(layer "Edge.Cuts")
+	)
+	(gr_line
+		(start 199.375 119.525)
+		(end 199.375 64.525)
+		(stroke
+			(width 0.0381)
+			(type solid)
+		)
 		(layer "Edge.Cuts")
 	)
 	(gr_line
 		(start 97.375 119.525)
-		(end 97.375 69.525)
+		(end 97.375 64.525)
 		(stroke
 			(width 0.0381)
@@
 		(polygon
 			(pts
-				(xy 95 67.85) (xy 95 121.85) (xy 201 121.85) (xy 201.1 67.25) (xy 95 67.25)
-			)
-		)
+				(xy 95 67.85) (xy 95 121.85) (xy 201 121.85) (xy 201.108789 62.45) (xy 95 62.45)
+			)
+		)
